File: Esp32_Modbus_Relay_hw/Esp32_Modbus_Relay_hw/Esp32_Modbus_Relay_hw.kicad_sch (KiCad schematic)
At the start: 70 parts, among them K1 SRA-5VDC-CL, Q1 2SC1815-HF, Q2 2SC1815/HF, U2 XL1509, U3 MAX485, U7 RT9193, U8 PC817

Commit message: Finish version 01
Parts:
- removed C5: 1uF_50V, Capacitor_SMD:C_0805_2012Metric_Pad1.18x1.45mm_HandSolder, symbol Device:C_Small
- removed L1: L_Ferrite, Inductor_THT:L_Radial_D6.0mm_P4.00mm, symbol Device:L_Ferrite
- removed U2: XL1509, Package_SO:SOIC-8-1EP_3.9x4.9mm_P1.27mm_EP2.41x3.81mm, symbol D_H_Lib_:XL1509
- removed U7: RT9193, Package_TO_SOT_SMD:SOT-23-5_HandSoldering, symbol ph_kicad_lib:RT9193
- added C28: 100nF, Capacitor_SMD:C_0805_2012Metric_Pad1.18x1.45mm_HandSolder, symbol library_by_DH:Capasitor_SMD
- added C31 (x12): 100nF, Capacitor_SMD:C_0805_2012Metric, symbol library_by_DH:Capasitor_SMD
- added C31: 1uF, Capacitor_SMD:C_0805_2012Metric, symbol library_by_DH:Capasitor_SMD
- added C34: 10uF, Capacitor_SMD:C_0805_2012Metric, symbol Device:C
- added C35: 100nF, Capacitor_SMD:C_0805_2012Metric, symbol Device:C
- added D12: 1N4007_T7, Diode_SMD:D_SOD-123F, symbol Device:D
- added J1: USB_C_Receptacle_USB2.0, Connector_USB:USB_C_Receptacle_GCT_USB4105-xx-A_16P_TopMnt_Horizontal, symbol Connector:USB_C_Receptacle_USB2.0
- added J2: UART0_EXT, Connector_PinHeader_2.54mm:PinHeader_1x04_P2.54mm_Vertical, symbol Connector:Conn_01x04_Pin
- added J3: header input, Lib_Hien:KF142_4P_5.08, symbol Connector:Conn_01x04_Pin
- added J4, J5: Conn_01x06_Pin, Lib_Hien:KF142_6P_5.08, symbol Connector:Conn_01x06_Pin
- added L3: 10uH, Inductor_SMD:L_0805_2012Metric, symbol Device:L_Ferrite
- added LED2: RED, LED_SMD:LED_0805_2012Metric_Pad1.15x1.40mm_HandSolder, symbol Device:LED
- added Q10, Q9: S8050, Package_TO_SOT_SMD:SOT-23, symbol Device:Q_NPN_BEC
- added Q8: 2SC1815-HF, Package_TO_SOT_SMD:SOT-23, symbol Device:Q_NPN_BEC
- added R17: 2.2K, Resistor_SMD:R_0805_2012Metric, symbol Device:R
- added R18, R21, R22, R23: 220R, Resistor_SMD:R_0805_2012Metric, symbol Device:R
- added R18 (x2): 10k, Resistor_SMD:R_0805_2012Metric, symbol Device:R
- added R18 (x2): 5.1K, Resistor_SMD:R_0805_2012Metric, symbol Device:R
- added R18 (x2): 470R, Resistor_SMD:R_0805_2012Metric, symbol Device:R
- added R22, R23, R36, R37, R38, R39, R40: 10K, Resistor_SMD:R_0805_2012Metric, symbol Device:R
- added R24: 1K, Resistor_SMD:R_0805_2012Metric_Pad1.20x1.40mm_HandSolder, symbol Device:R
- added SW1, SW2, SW3, SW4, SW5, SW6: SW_Push, Button_Switch_SMD:SW_DIP_SPSTx01_Slide_6.7x4.1mm_W8.61mm_P2.54mm_LowProfile, symbol Switch:SW_Push
- added U1: AMS1117-3.3, Package_TO_SOT_SMD:SOT-223-3_TabPin2, symbol Regulator_Linear:AMS1117-3.3
- added U11: CP2102-GM, Lib_Hien:CP2102, symbol lib_Hien:CP2102
- added U9: 2.2inch_TFT_ILI9341_SPI, Lib_Hien:TFT_ILI9341_2.2INCH, symbol Lib_Mr_DH:2.2inch_TFT_ILI9341_SPI
- added V1, V2, V3, V4: Vit, Lib_Hien:Vit, symbol lib_Hien:Vit
- added VR1: LM2596S-ADJ, Lib_Hien:LM2596S-ADJ, symbol Lib_Hien:LM2596S-ADJ
- C31, C32: footprint Capacitor_SMD:C_0805_2012Metric_Pad1.18x1.45mm_HandSolder -> Capacitor_SMD:C_0805_2012Metric
- C6: value 220uF_50V -> 470uF/25V; footprint Capacitor_SMD:CP_Elec_8x10.5 -> Capacitor_SMD:CP_Elec_10x10
- C8: value 180uF_35v -> 220uF/25V; footprint Capacitor_SMD:CP_Elec_6.3x9.9 -> Capacitor_SMD:CP_Elec_8x10.5
- D2: value 1N4007_M7 -> ES3J_3A; footprint Diode_SMD:D_SMA -> Diode_SMD:D_SMC
- F1: value Polyfuse -> UF300_3A; footprint Fuse:Fuse_1812_4532Metric_Pad1.30x3.40mm_HandSolder -> Fuse:Fuse_BelFuse_0ZRE0033FF_L11.4mm_W3.8mm
- F2, F3: footprint Fuse:Fuse_1812_4532Metric_Pad1.30x3.40mm_HandSolder -> Lib_Hien:Fuse_SMD_1812
- L2: value 68uH_2A -> 33uH_2.9A; footprint Inductor_SMD:L_Bourns-SRU8028_8.0x8.0mm -> Lib_Hien:L_10x10
Connections:
- net Earth is gone; now on net GND: C6.2, C7.2, C8.2, C9.1, D1.1 (A1), D3.2 (A), D4.2 (A2), D5.1 (A1), Q1.2 (E), R1.1, R8.2, U3.4 (DI), U3.5 (GND)
- net UART0_RX is gone; now on net RXD1: R1.2, R2.1
- net UART0_TX is gone; now on net TXD1: R3.1
- net +12V: now also J3.1 (Pin_1)
- net +3.3V: now also C31.1, C31.1, C31.1, C34.1, C35.1, J2.1 (Pin_1), L3.2, R22.1, R23.1, R24.1, R36.1, R37.1, R38.1, R39.1, R40.1, U1.2 (VO), U11.6 (VDD), U11.7 (REGIN), U9.10 (LEDA), U9.9 (VCC)
- net +5V: now also C28.1, C31.1, C31.1, D12.1 (K), U1.3 (VI), U11.8 (VBUS), VR1.4 (FB)
- net A: now also J3.3 (Pin_3)
- net B: now also J3.4 (Pin_4)
- net COM1: now also J4.1 (Pin_1)
- net COM2: now also J4.3 (Pin_3)
- net COM3: now also J4.5 (Pin_5)
- net COM4: now also J5.1 (Pin_1)
- net COM5: now also J5.3 (Pin_3)
- net COM6: now also J5.5 (Pin_5)
- net DO1: now also A1.14 (IO12)
- net DO2: now also A1.16 (IO13)
- net DO3: now also A1.13 (IO14)
- net DO4: now also A1.12 (IO27)
- net DO5: now also A1.10 (IO25)
- net DO6: now also A1.11 (IO26)
- net GND: now also A1.1 (GND), A1.15 (GND), A1.38 (GND), C28.2, C31.2, C31.2, C31.2, C31.2, C31.2, C31.2, C31.2, C31.2, C31.2, C31.2, C31.2, C31.2, C31.2, C34.2, C35.2, J1.A1 (GND), J1.A12 (GND), J1.A8 (SBU1), J1.B1 (GND), J1.B12 (GND), J1.B8 (SBU2), J1.S1 (SHIELD), J2.4 (Pin_4), J3.2 (Pin_2), Q8.2 (E), R18.1, R18.1, SW1.2, SW2.2, SW3.2, SW4.2, SW5.2, SW6.2, U1.1 (GND), U11.29 (GND), U11.3 (GND), U9.1 (GND), U9.2 (RESET), U9.8 (GND), VR1.3 (GND), VR1.5 (~{ON}/OFF), VR1.6 (GND)
- net NO1: now also J4.2 (Pin_2)
- net NO2: now also J4.4 (Pin_4)
- net NO3: now also J4.6 (Pin_6)
- net NO4: now also J5.2 (Pin_2)
- net NO5: now also J5.4 (Pin_4)
- net NO6: now also J5.6 (Pin_6)
- net at D2.1 (K): now also C6.1, C7.1, VR1.1 (VIN)
- net at D3.1 (K), L2.1: now also VR1.2 (OUT)
- net at A1.2 (VDD3V3): now also C31.1, L3.1
- net DOWN: now reaches A1.23 (IO15)
- net DOWN: now also C31.1, R37.2, SW3.1
- net UP: now reaches A1.24 (IO2)
- net UP: now also C31.1, R36.2, SW2.1
- net BOOT: now reaches A1.25 (IO0)
- net BOOT: now also C31.1, Q10.3 (C), R23.2, SW1.1
- net Blink: now reaches A1.26 (IO4)
- net Blink: now also LED2.1 (K)
- net OK: now reaches A1.29 (IO5)
- net OK: now also C31.1, R40.2, SW6.1
- net EN: now reaches A1.3 (EN)
- net EN: now also C31.1, Q9.3 (C), R22.2
- net LEFT: now reaches A1.30 (IO18)
- net LEFT: now also C31.1, R38.2, SW4.1
- net RIGHT: now reaches A1.31 (IO19)
- net RIGHT: now also C31.1, R39.2, SW5.1
- net LCD_MISO: now reaches A1.33 (IO21)
- net LCD_MISO: now also U9.7 (SD0)
- net RXD0: now reaches A1.34 (RXD0)
- net RXD0: now also J2.2 (Pin_2), R18.1
- net TXD0: now reaches A1.35 (TXD0)
- net TXD0: now also J2.3 (Pin_3), R18.1
- net TXD1: now reaches A1.36 (IO22)
- net RXD1: now reaches A1.37 (IO23)
- net LCD_BL: now reaches A1.4 (SENSOR_VP)
- net LCD_BL: now also R17.1
- net GPIO36/ADC1_CH0: now reaches A1.5 (SENSOR_VN)
- net LCD_DC: now reaches A1.6 (IO34)
- net LCD_DC: now also U9.4 (D/C)
- net LCD_SCL: now reaches A1.7 (IO35)
- net LCD_SCL: now also U9.3 (SCL)
- net LCD_MOSI: now reaches A1.8 (IO32)
- net LCD_MOSI: now also U9.6 (SDA)
- net LCD_CS0: now reaches A1.9 (IO33)
- net LCD_CS0: now also U9.5 (CS)
- new net: Q8.3 (C), R18.1, R21.1, R22.1, R23.1
- new net: Q8.1 (B), R17.2
- new net: Q9.1 (B), R18.1
- new net: J1.B5 (CC2), R18.2
- new net: Q10.1 (B), R18.1
- new net: LED2.2 (A), R24.2
- new net: D12.2 (A), J1.A4 (VBUS), J1.A9 (VBUS), J1.B4 (VBUS), J1.B9 (VBUS)
- new net: J1.A5 (CC1), R18.2
- new net BL1-: R18.2, U9.11 (LEDK1)
- new net BL2-: R21.2, U9.12 (LEDK2)
- new net BL3-: R22.2, U9.13 (LEDK3)
- new net BL4-: R23.2, U9.14 (LEDK4)
- new net CP_CTS: U11.23 (~{CTS})
- new net CP_DCD: U11.1 (~{DCD})
- new net CP_DSR: U11.27 (~{DSR})
- new net CP_DTR: Q10.2 (E), R18.2, U11.28 (~{DTR})
- new net CP_RI: U11.2 (~{RI})
- new net CP_RST: Q9.2 (E), R18.2, U11.24 (~{RST})
- new net CP_RXD: R18.2, U11.25 (RXD)
- new net CP_TXD: R18.2, U11.26 (TXD)
- new net USB_D+: J1.A6 (D+), J1.B6 (D+), U11.4 (D+)
- new net USB_D-: J1.A7 (D-), J1.B7 (D-), U11.5 (D–)
- new net X+: U9.17 (XR)
- new net X-: U9.15 (XL)
- new net Y+: U9.18 (YD)
- new net Y-: U9.16 (YU)
- no-connect marks 0 -> 11
Other:
- note added: "5VDC TO 3.3VDC"
- note added: "BUTTON INPUT"
- note added: "LCD 2.2Inch TFT-ILI9341"
- note added: "MCU ESP32-WROVER-B"
- note added: "MODBUS RTU"
- note added: "POWER 12V INPUT"
- note added: "RELAY CONTROL"
- note added: "USB-C"
- note removed: "MAX485 (MODBUS)"
- moved on the sheet: A1, C28, C29, C31, C32, C6, C7, C8, C9, D1, D2, D3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
